File: mic.sch (EAGLE design)
At the start: 10 parts, among them IC1 AD8614RJ, M1 ELECTRET_MICROPHON-WM.64PN

Commit message: Breakout board and PNGs for electret mic circuit.
Parts:
- removed M1: ELECTRET_MICROPHON-WM.64PN, microphon:ELECTRET_MICROPHON-WM.64PN
- added U$1: ELECTRET, LED Light:ELECTRET
Connections:
- net GND: now also U$1.2; no longer M1.2
- net N$4: now also U$1.1; no longer M1.1
Changed lines of the file:
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@@
 <layer number="48" name="Document" color="7" fill="1" visible="no" active="no"/>
 <layer number="49" name="Reference" color="7" fill="1" visible="no" active="no"/>
+<layer number="50" name="dxf" color="7" fill="1" visible="no" active="no"/>
 <layer number="51" name="tDocu" color="7" fill="1" visible="no" active="no"/>
 <layer number="52" name="bDocu" color="7" fill="1" visible="no" active="no"/>
+<layer number="53" name="tGND_GNDA" color="7" fill="9" visible="no" active="no"/>
+<layer number="54" name="bGND_GNDA" color="1" fill="9" visible="no" active="no"/>
+<layer number="56" name="wert" color="7" fill="1" visible="no" active="no"/>
 <layer number="91" name="Nets" color="2" fill="1" visible="yes" active="yes"/>
 <layer number="92" name="Busses" color="1" fill="1" visible="yes" active="yes"/>
@@
 <layer number="97" name="Info" color="7" fill="1" visible="yes" active="yes"/>
 <layer number="98" name="Guide" color="6" fill="1" visible="yes" active="yes"/>
+<layer number="100" name="Muster" color="7" fill="1" visible="no" active="no"/>
+<layer number="101" name="Patch_Top" color="12" fill="4" visible="no" active="yes"/>
+<layer number="102" name="Vscore" color="7" fill="1" visible="no" active="yes"/>
+<layer number="104" name="Name" color="7" fill="1" visible="no" active="yes"/>
+<layer number="116" name="Patch_BOT" color="9" fill="4" visible="no" active="yes"/>
+<layer number="121" name="_tsilk" color="7" fill="1" visible="no" active="yes"/>
+<layer number="122" name="_bsilk" color="7" fill="1" visible="no" active="yes"/>
+<layer number="151" name="HeatSink" color="7" fill="1" visible="no" active="yes"/>
+<layer number="200" name="200bmp" color="1" fill="10" visible="no" active="yes"/>
+<layer number="201" name="201bmp" color="2" fill="10" visible="no" active="yes"/>
+<layer number="202" name="202bmp" color="3" fill="10" visible="no" active="yes"/>
+<layer number="203" name="203bmp" color="4" fill="10" visible="no" active="yes"/>
+<layer number="204" name="204bmp" color="5" fill="10" visible="no" active="yes"/>
+<layer number="205" name="205bmp" color="6" fill="10" visible="no" active="yes"/>
+<layer number="206" name="206bmp" color="7" fill="10" visible="no" active="yes"/>
+<layer number="207" name="207bmp" color="8" fill="10" visible="no" active="yes"/>
+<layer number="208" name="208bmp" color="9" fill="10" visible="no" active="yes"/>
+<layer number="250" name="Descript" color="3" fill="1" visible="no" active="no"/>
+<layer number="251" name="SMDround" color="12" fill="11" visible="no" active="no"/>
+<layer number="254" name="cooling" color="7" fill="1" visible="no" active="yes"/>
 </layers>
 <schematic xreflabel="%F%N/%S.%C%R" xrefpart="/%S.%C%R">
@@
 <part name="R2" library="rcl" deviceset="R-US_" device="R1206" value="10K"/>
 <part name="C1" library="rcl" deviceset="C-US" device="C1206" value="0.1uF"/>
-<part name="M1" library="microphon" deviceset="ELECTRET_MICROPHON-" device="WM.64PN"/>
 <part name="R3" library="rcl" deviceset="R-US_" device="R1206" value="10K"/>
 <part name="R4" library="rcl" deviceset="R-US_" device="R1206" value="10K"/>
 <part name="C2" library="rcl" deviceset="C-US" device="C1206" value="1uF"/>
 <part name="R5" library="rcl" deviceset="R-US_" device="R1206" value="1K"/>
+<part name="U$1" library="LED Light" deviceset="ELECTRET" device=""/>
 </parts>
 <sheets>
@@
 <instance part="R2" gate="G$1" x="40.64" y="53.34" rot="R90"/>
 <instance part="C1" gate="G$1" x="25.4" y="58.42"/>
-<instance part="M1" gate="G$1" x="114.3" y="55.88"/>
 <instance part="R3" gate="G$1" x="78.74" y="55.88"/>
 <instance part="R4" gate="G$1" x="109.22" y="60.96" rot="R90"/>
 <instance part="C2" gate="G$1" x="99.06" y="55.88" rot="R90"/>
 <instance part="R5" gate="G$1" x="91.44" y="55.88"/>
+<instance part="U$1" gate="G$1" x="116.84" y="55.88"/>
 </instances>
 <busses>
@@
 </segment>
 <segment>
-<pinref part="M1" gate="G$1" pin="2"/>
 <wire x1="109.22" y1="53.34" x2="109.22" y2="40.64" width="0.1524" layer="91"/>
 <label x="106.68" y="38.1" size="1.778" layer="95"/>
+<pinref part="U$1" gate="G$1" pin="2"/>
 </segment>
 <segment>
@@
 <net name="N$4" class="0">
 <segment>
-<pinref part="M1" gate="G$1" pin="1"/>
 <pinref part="R4" gate="G$1" pin="1"/>
 <pinref part="C2" gate="G$1" pin="2"/>
@@
 <pinref part="C2" gate="G$1" pin="2"/>
 <wire x1="104.14" y1="55.88" x2="109.22" y2="55.88" width="0.1524" layer="91"/>
+<pinref part="U$1" gate="G$1" pin="1"/>
 <junction x="109.22" y="55.88"/>
 </segment>
